Commit message: migrating to python

File: +scara0/model.urdf (robot description, URDF)
Before this commit: robot scara_robot, 4 links, 3 joints
Links:
- added link flange
- link link1: geometry visual cylinder length=0.4 radius=0.05
- link link2: geometry visual cylinder length=0.4 radius=0.05
Joints:
- added joint joint_flange: type fixed, parent link2, child flange, origin xyz=0.4 0 0 rpy=0 0 0
- joint joint2: origin xyz=0.3 0 0 rpy=0 0 0 -> xyz=0.4 0 0 rpy=0 0 0
